File: ulp.kicad_pcb (KiCad board)
At the start: 2 copper layers, 102 x 84.2 mm, 50 parts, among them J1 Conn_01x01_Pin, J2 Conn_01x01_Pin, SW1 SW_Push_45deg, SW10 SW_Push_45deg, SW11 SW_Push_45deg, SW12 SW_Push_45deg, SW13 SW_Push_45deg, SW14 SW_Push_45deg, SW15 SW_Push_45deg, SW16 SW_Push_45deg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

Commit message: small changes
Routing:
- removed copper zone on B.Cu, net GND
- removed copper zone on F.Cu, net GND
Changed lines of the file:
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@@
 		)
 		(pad "3" smd rect
-			(at -6.200002 5.025 9)
+			(at -6.200003 5.025 9)
 			(size 1.6 1.8)
 			(layers "F.Cu" "F.Mask" "F.Paste")
 		)
 		(pad "3" smd rect
-			(at -6.200002 5.025 9)
+			(at -6.200003 5.025 9)
 			(size 1.6 1.8)
 			(layers "B.Cu" "B.Mask" "B.Paste")
@@
 		)
 		(pad "3" smd rect
-			(at 6.200002 -5.025 9)
+			(at 6.200003 -5.025 9)
 			(size 1.6 1.8)
 			(layers "F.Cu" "F.Mask" "F.Paste")
 		)
 		(pad "3" smd rect
-			(at 6.200002 -5.025 9)
+			(at 6.200003 -5.025 9)
 			(size 1.6 1.8)
 			(layers "B.Cu" "B.Mask" "B.Paste")
@@
 		(fp_line
 			(start -0.465003 0)
-			(end 0.332138 -0.531434)
+			(end 0.332137 -0.531434)
 			(stroke
 				(width 0.132857)
@@
 		)
 		(fp_line
-			(start 0.332138 -0.531434)
+			(start 0.332137 -0.531434)
 			(end 0.33214 0.531434)
 			(stroke
@@
 		)
 		(fp_line
-			(start -0.332138 0.531434)
+			(start -0.332137 0.531434)
 			(end -0.33214 -0.531434)
 			(stroke
@@
 		(fp_line
 			(start 0.465003 0)
-			(end -0.332138 0.531434)
+			(end -0.332137 0.531434)
 			(stroke
 				(width 0.132857)
@@
 		(fp_line
 			(start -0.465003 0)
-			(end 0.332138 -0.531434)
+			(end 0.332137 -0.531434)
 			(stroke
 				(width 0.132857)
@@
 		)
 		(fp_line
-			(start 0.332138 -0.531434)
+			(start 0.332137 -0.531434)
 			(end 0.33214 0.531434)
 			(stroke
@@
 		)
 		(pad "3" smd rect
-			(at -6.200002 5.025 9)
+			(at -6.200003 5.025 9)
 			(size 1.6 1.8)
 			(layers "F.Cu" "F.Mask" "F.Paste")
 		)
 		(pad "3" smd rect
-			(at -6.200002 5.025 9)
+			(at -6.200003 5.025 9)
 			(size 1.6 1.8)
 			(layers "B.Cu" "B.Mask" "B.Paste")
@@
 		)
 		(pad "3" smd rect
-			(at 6.200002 -5.025 9)
+			(at 6.200003 -5.025 9)
 			(size 1.6 1.8)
 			(layers "F.Cu" "F.Mask" "F.Paste")
 		)
 		(pad "3" smd rect
-			(at 6.200002 -5.025 9)
+			(at 6.200003 -5.025 9)
 			(size 1.6 1.8)
 			(layers "B.Cu" "B.Mask" "B.Paste")
@@
 		)
 		(pad "3" smd rect
-			(at -6.200002 5.025 9)
+			(at -6.200003 5.025 9)
 			(size 1.6 1.8)
 			(layers "F.Cu" "F.Mask" "F.Paste")
 		)
 		(pad "3" smd rect
-			(at -6.200002 5.025 9)
+			(at -6.200003 5.025 9)
 			(size 1.6 1.8)
 			(layers "B.Cu" "B.Mask" "B.Paste")
@@
 		)
 		(pad "3" smd rect
-			(at 6.200002 -5.025 9)
+			(at 6.200003 -5.025 9)
 			(size 1.6 1.8)
 			(layers "F.Cu" "F.Mask" "F.Paste")
 		)
 		(pad "3" smd rect
-			(at 6.200002 -5.025 9)
+			(at 6.200003 -5.025 9)
 			(size 1.6 1.8)
 			(layers "B.Cu" "B.Mask" "B.Paste")
@@
 		(net "Net-(D8-A)")
 	)
-	(zone
-		(net "GND")
-		(layers "F.Cu" "B.Cu")
-		(hatch edge 0.5)
-		(connect_pads
-			(clearance 0.5)
-		)
-		(min_thickness 0.25)
-		(fill yes
-			(thermal_gap 0.5)
-			(thermal_bridge_width 0.5)
-			(island_removal_mode 0)
-		)
-		(polygon
-			(pts
-				(xy 92.507903 50.129398) (xy 212.507903 50.129398) (xy 212.507903 147.629398) (xy 92.507903 150.129398)
-			)
-		)
-	)
 	(embedded_fonts no)
