File: ulp.kicad_pcb (KiCad board)
At the start: 2 copper layers, 102 x 84.2 mm, 50 parts, among them J1 Conn_01x01_Pin, J2 Conn_01x01_Pin, SW1 SW_Push_45deg, SW10 SW_Push_45deg, SW11 SW_Push_45deg, SW12 SW_Push_45deg, SW13 SW_Push_45deg, SW14 SW_Push_45deg, SW15 SW_Push_45deg, SW16 SW_Push_45deg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

Commit message: Stop tracking ignored files
Amp-Thread-ID: https://ampcode.com/threads/T-019e7445-9c97-7198-8a44-fdf52582fa4e
Co-authored-by: Amp <amp@ampcode.com>
Routing:
- net GND: vias 1 -> 2
- added copper zone on B.Cu, net GND
- added copper zone on F.Cu, net GND
Other:
- board text added: "BATT+"
Changed lines of the file:
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@@
 		(capping no)
 		(filling no)
-		(grid_origin 109.965753 59.547521)
+		(grid_origin 113.091819 64.014801)
 		(pcbplotparams
 			(layerselection 0x00000000_00000000_55555555_5755f5ff)
@@
 	)
 	(gr_rect
-		(start 106.415752 58.572522)
-		(end 108.165649 59.39774)
+		(start 113.091819 64.264801)
+		(end 114.591818 65.814801)
+		(stroke
+			(width 0.1)
+			(type solid)
+		)
+		(fill yes)
+		(layer "F.SilkS")
+	)
+	(gr_rect
+		(start 102.606321 64.289801)
+		(end 104.10632 65.839801)
 		(stroke
 			(width 0.1)
@@
 	)
 	(gr_rect
-		(start 137.257903 13.879398)
-		(end 187.257903 44.379398)
+		(start 106.415752 58.572522)
+		(end 108.165649 59.39774)
 		(stroke
 			(width 0.1)
 			(type solid)
 		)
-		(fill no)
-		(layer "Dwgs.User")
+		(fill yes)
+		(layer "B.SilkS")
 	)
 	(gr_line
@@
 		)
 	)
+	(gr_text "BATT+"
+		(at 114.641819 64.264801 90)
+		(layer "F.SilkS")
+		(effects
+			(font
+				(size 1.1 1.1)
+				(thickness 0.25)
+				(bold yes)
+			)
+			(justify left bottom)
+		)
+	)
 	(gr_text "+"
 		(at 107.090753 59.322521 45)
@@
 		)
 	)
+	(gr_text "BATT+"
+		(at 102.55632 64.289801 -90)
+		(layer "B.SilkS")
+		(effects
+			(font
+				(size 1.1 1.1)
+				(thickness 0.25)
+				(bold yes)
+			)
+			(justify left bottom mirror)
+		)
+	)
 	(gr_text "RST\n"
 		(at 106.540753 58.397521 -90)
@@
 	)
 	(via
+		(at 197.041819 61.564801)
+		(size 0.6)
+		(drill 0.3)
+		(layers "F.Cu" "B.Cu")
+		(free yes)
+		(net "GND")
+	)
+	(via
 		(at 108.615753 73.597521)
 		(size 0.7)
@@
 		(net "Net-(D8-A)")
 	)
+	(zone
+		(net "GND")
+		(layers "F.Cu" "B.Cu")
+		(hatch edge 0.5)
+		(connect_pads
+			(clearance 0.5)
+		)
+		(min_thickness 0.25)
+		(fill yes
+			(thermal_gap 0.5)
+			(thermal_bridge_width 0.5)
+			(island_removal_mode 0)
+		)
+		(polygon
+			(pts
+				(xy 200.641819 54.764801) (xy 200.641819 138.964802) (xy 98.641818 138.964802) (xy 98.641818 54.764801)
+			)
+		)
+	)
 	(embedded_fonts no)

Commit message: update pcb
Parts:
- removed the J1 at (173.3, 58.6)
- removed the J2 at (173.3, 61.4)
- added C1: C_Small, reversible:C_0603_1608Metric_Reversible, F.Cu at (193.1, 61.9)
- D1, D10, D11, D12, D13, D14, D15, D16, D17, D18, D2, D3, D4, D5, D6, D7, D8, D9: footprint reversible:D_SOD-123 -> reversible:D_SOD-123_Reversible
- D19: footprint reversible:led reversible -> reversible:LED_WS2812B_PLCC4_5.0x5.0mm_P3.2mm_Reversible
- J1, J2: footprint Connector_Wire:SolderWirePad_1x01_SMD_2x4mm -> reversible:TestPoint_Pad_2.0x4.0mm_Reversible
- SW19: footprint switches:power_switch -> reversible:SW_SPDT_MSK-12C02_Reversible
- SW20: footprint switches:reset_switch -> reversible:SW_Push_SPST_EVQ-PU_Reversible
- U2: footprint reversible handsolder xiao nrf:XIAO-nRF52840-handsolder -> reversible:MODULE_Seeed_XIAO_nRF52840_THT_Reversible
Routing:
- net GND: track 10.9 -> 19.5 mm
- net +5V: track 94.6 -> 99.3 mm, vias 2 -> 3
- net /column 4: track 176.5 -> 178.0 mm

Commit message: add .step files of each side
Routing:
- net GND: track 19.5 -> 15.9 mm
- net /BATT_RAW: track 18.0 -> 17.4 mm
