File: ulp.kicad_sch (KiCad schematic)
At the start: 49 parts, among them J1 Conn_01x01_Pin, J2 Conn_01x01_Pin, SW1 SW_Push_45deg, SW10 SW_Push_45deg, SW11 SW_Push_45deg, SW12 SW_Push_45deg, SW13 SW_Push_45deg, SW14 SW_Push_45deg, SW15 SW_Push_45deg, SW16 SW_Push_45deg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

Commit message: update pcb
Parts:
- C1: footprint (none) -> reversible:C_0603_1608Metric_Reversible
- D1, D10, D11, D12, D13, D14, D15, D16, D17, D18, D2, D3, D4, D5, D6, D7, D8, D9: footprint reversible:D_SOD-123 -> reversible:D_SOD-123_Reversible
- D19: footprint reversible:led reversible -> reversible:LED_WS2812B_PLCC4_5.0x5.0mm_P3.2mm_Reversible
- J1, J2: footprint Connector_Wire:SolderWirePad_1x01_SMD_2x4mm -> reversible:TestPoint_Pad_2.0x4.0mm_Reversible
- SW19: footprint switches:power_switch -> reversible:SW_SPDT_MSK-12C02_Reversible
- SW20: footprint switches:reset_switch -> reversible:SW_Push_SPST_EVQ-PU_Reversible
- U2: footprint reversible handsolder xiao nrf:XIAO-nRF52840-handsolder -> reversible:MODULE_Seeed_XIAO_nRF52840_THT_Reversible
Changed lines of the file:
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@@
 	(wire
 		(pts
-			(xy 151.13 45.72) (xy 161.29 45.72)
+			(xy 151.13 53.34) (xy 161.29 53.34)
 		)
 		(stroke
@@
 	(wire
 		(pts
-			(xy 151.13 53.34) (xy 161.29 53.34)
+			(xy 151.13 45.72) (xy 161.29 45.72)
 		)
 		(stroke
@@
 	(wire
 		(pts
+			(xy 151.13 57.15) (xy 161.29 57.15)
+		)
+		(stroke
+			(width 0)
+			(type default)
+		)
+	)
+	(wire
+		(pts
 			(xy 24.13 59.69) (xy 36.83 59.69)
 		)
@@
 	(wire
 		(pts
-			(xy 151.13 57.15) (xy 161.29 57.15)
-		)
-		(stroke
-			(width 0)
-			(type default)
-		)
-	)
-	(wire
-		(pts
 			(xy 135.89 101.6) (xy 139.7 101.6)
 		)
@@
 	(wire
 		(pts
-			(xy 62.23 90.17) (xy 74.93 90.17)
-		)
-		(stroke
-			(width 0)
-			(type default)
-		)
-	)
-	(wire
-		(pts
-			(xy 149.86 118.11) (xy 153.67 118.11)
+			(xy 151.13 38.1) (xy 152.4 38.1)
 		)
 		(stroke
@@
 	(wire
 		(pts
-			(xy 57.15 34.29) (xy 57.15 49.53)
+			(xy 62.23 90.17) (xy 74.93 90.17)
 		)
 		(stroke
@@
 	(wire
 		(pts
-			(xy 31.75 110.49) (xy 31.75 115.57)
+			(xy 149.86 118.11) (xy 153.67 118.11)
 		)
 		(stroke
@@
 	(wire
 		(pts
-			(xy 151.13 41.91) (xy 154.94 41.91)
+			(xy 57.15 34.29) (xy 57.15 49.53)
 		)
 		(stroke
@@
 	(wire
 		(pts
-			(xy 151.13 49.53) (xy 161.29 49.53)
+			(xy 31.75 110.49) (xy 31.75 115.57)
 		)
 		(stroke
@@
 	(wire
 		(pts
-			(xy 151.13 38.1) (xy 152.4 38.1)
+			(xy 151.13 41.91) (xy 154.94 41.91)
 		)
 		(stroke
@@
 	(wire
 		(pts
+			(xy 151.13 49.53) (xy 161.29 49.53)
+		)
+		(stroke
+			(width 0)
+			(type default)
+		)
+	)
+	(wire
+		(pts
 			(xy 133.35 19.05) (xy 133.35 22.86)
 		)
@@
 			)
 		)
-		(property "Footprint" "reversible:D_SOD-123"
+		(property "Footprint" "reversible:D_SOD-123_Reversible"
 			(at 49.53 57.15 90)
 			(hide yes)
@@
 			)
 		)
-		(property "Footprint" "reversible:D_SOD-123"
+		(property "Footprint" "reversible:D_SOD-123_Reversible"
 			(at 36.83 41.91 90)
 			(hide yes)
@@
 			)
 		)
-		(property "Footprint" "reversible:D_SOD-123"
+		(property "Footprint" "reversible:D_SOD-123_Reversible"
 			(at 24.13 41.91 90)
 			(hide yes)
@@
 			)
 		)
-		(property "Footprint" "reversible handsolder xiao nrf:XIAO-nRF52840-handsolder"
+		(property "Footprint" "reversible:MODULE_Seeed_XIAO_nRF52840_THT_Reversible"
 			(at 121.92 40.64 0)
 			(hide yes)
@@
 			)
 		)
-		(property "Footprint" "Connector_Wire:SolderWirePad_1x01_SMD_2x4mm"
+		(property "Footprint" "reversible:TestPoint_Pad_2.0x4.0mm_Reversible"
 			(at 81.915 107.95 0)
 			(hide yes)
@@
 			)
 		)
-		(property "Footprint" "reversible:D_SOD-123"
+		(property "Footprint" "reversible:D_SOD-123_Reversible"
 			(at 62.23 72.39 90)
 			(hide yes)
@@
 			)
 		)
-		(property "Footprint" "reversible:D_SOD-123"
+		(property "Footprint" "reversible:D_SOD-123_Reversible"
 			(at 24.13 72.39 90)
 			(hide yes)
@@
 			)
 		)
-		(property "Footprint" "reversible:D_SOD-123"
+		(property "Footprint" "reversible:D_SOD-123_Reversible"
 			(at 74.93 87.63 90)
 			(hide yes)
@@
 			)
 		)
-		(property "Footprint" "reversible:D_SOD-123"
+		(property "Footprint" "reversible:D_SOD-123_Reversible"
 			(at 74.93 41.91 90)
 			(hide yes)
@@
 			)
 		)
-		(property "Footprint" "switches:power_switch"
+		(property "Footprint" "reversible:SW_SPDT_MSK-12C02_Reversible"
 			(at 53.34 111.76 0)
 			(hide yes)
@@
 			)
 		)
-		(property "Footprint" "switches:reset_switch"
+		(property "Footprint" "reversible:SW_Push_SPST_EVQ-PU_Reversible"
 			(at 25.4 105.41 0)
 			(hide yes)
@@
 			)
 		)
-		(property "Footprint" "reversible:led reversible"
+		(property "Footprint" "reversible:LED_WS2812B_PLCC4_5.0x5.0mm_P3.2mm_Reversible"
 			(at 109.22 107.95 0)
 			(hide yes)
@@
 			)
 		)
-		(property "Footprint" "reversible:D_SOD-123"
+		(property "Footprint" "reversible:D_SOD-123_Reversible"
 			(at 36.83 57.15 90)
 			(hide yes)
@@
 			)
 		)
-		(property "Footprint" "reversible:D_SOD-123"
+		(property "Footprint" "reversible:D_SOD-123_Reversible"
 			(at 74.93 72.39 90)
 			(hide yes)
@@
 			)
 		)
-		(property "Footprint" "reversible:D_SOD-123"
+		(property "Footprint" "reversible:D_SOD-123_Reversible"
 			(at 36.83 72.39 90)
 			(hide yes)
@@
 			)
 		)
-		(property "Footprint" "reversible:D_SOD-123"
+		(property "Footprint" "reversible:D_SOD-123_Reversible"
 			(at 62.23 57.15 90)
 			(hide yes)
@@
 			)
 		)
-		(property "Footprint" "reversible:D_SOD-123"
+		(property "Footprint" "reversible:D_SOD-123_Reversible"
 			(at 62.23 87.63 90)
 			(hide yes)
@@
 			)
 		)
-		(property "Footprint" "reversible:D_SOD-123"
+		(property "Footprint" "reversible:D_SOD-123_Reversible"
 			(at 49.53 72.39 90)
 			(hide yes)
@@
 			)
 		)
-		(property "Footprint" "reversible:D_SOD-123"
+		(property "Footprint" "reversible:D_SOD-123_Reversible"
 			(at 49.53 87.63 90)
 			(hide yes)
@@
 			)
 		)
-		(property "Footprint" "reversible:D_SOD-123"
+		(property "Footprint" "reversible:D_SOD-123_Reversible"
 			(at 74.93 57.15 90)
 			(hide yes)
@@
 			)
 		)
-		(property "Footprint" "reversible:D_SOD-123"
+		(property "Footprint" "reversible:D_SOD-123_Reversible"
 			(at 24.13 57.15 90)
 			(hide yes)
@@
 			)
 		)
-		(property "Footprint" "Connector_Wire:SolderWirePad_1x01_SMD_2x4mm"
+		(property "Footprint" "reversible:TestPoint_Pad_2.0x4.0mm_Reversible"
 			(at 77.47 116.84 0)
 			(hide yes)
@@
 			)
 		)
-		(property "Footprint" ""
+		(property "Footprint" "reversible:C_0603_1608Metric_Reversible"
 			(at 125.73 100.33 0)
 			(hide yes)
@@
 			)
 		)
-		(property "Footprint" "reversible:D_SOD-123"
+		(property "Footprint" "reversible:D_SOD-123_Reversible"
 			(at 49.53 41.91 90)
 			(hide yes)
@@
 			)
 		)
-		(property "Footprint" "reversible:D_SOD-123"
+		(property "Footprint" "reversible:D_SOD-123_Reversible"
 			(at 62.23 41.91 90)
 			(hide yes)

Commit message: add mounting holes and new models
Parts:
- added H1, H2, H3, H4: MountingHole, MountingHole:MountingHole_2.2mm_M2, symbol Mechanical:MountingHole
